Commit message: Adding Gazebo Control

File: description/robot.urdf.xacro (robot description, xacro)
@@ -2,3 +2,4 @@
 <robot xmlns:xacro="http://www.ros.org/wiki/xacro"  name="spd">
     <xacro:include filename="robot_core.xacro"/>
+    <xacro:include filename="gazebo_control.xacro"/>
 </robot>

File: description/robot_core.xacro (robot description, xacro)
@@ -17,5 +17,5 @@
     <!-- BASE LINK -->
     <link name="base_link"></link>
-    <!-- BASE_FOOTPRINT LINK -->
+    <!-- BASE FOOTPRINT LINK -->
     <joint name="base_footprint_joint" type="fixed">
         <parent link="base_link"/>
@@ -103,12 +103,12 @@
         <material>Gazebo/Yellow</material>
     </gazebo>
-    <!-- BACK LEFT WHEEL LINK -->
-    <joint name="back_left_wheel_joint" type="continuous">
+    <!-- REAR LEFT WHEEL LINK -->
+    <joint name="rear_left_wheel_joint" type="continuous">
         <parent link="base_link"/>
-        <child link="back_left_wheel"/>
+        <child link="rear_left_wheel"/>
         <origin xyz="${-wheel_offset_x} ${wheel_offset_y} 0" rpy="-${pi/2} 0 0" />
         <axis xyz="0 0 1"/>
     </joint>
-    <link name="back_left_wheel">
+    <link name="rear_left_wheel">
         <visual>
             <geometry>
@@ -126,15 +126,15 @@
         </xacro:inertial_cylinder>
     </link>
-    <gazebo reference="back_left_wheel">
+    <gazebo reference="rear_left_wheel">
         <material>Gazebo/Yellow</material>
     </gazebo>
-    <!-- BACK RIGHT WHEEL LINK -->
-    <joint name="back_right_wheel_joint" type="continuous">
+    <!-- REAR RIGHT WHEEL LINK -->
+    <joint name="rear_right_wheel_joint" type="continuous">
         <parent link="base_link"/>
-        <child link="back_right_wheel"/>
+        <child link="rear_right_wheel"/>
         <origin xyz="${-wheel_offset_x} ${-wheel_offset_y} 0" rpy="${pi/2} 0 0" />
         <axis xyz="0 0 -1"/>
     </joint>
-    <link name="back_right_wheel">
+    <link name="rear_right_wheel">
         <visual>
             <geometry>
@@ -152,5 +152,5 @@
         </xacro:inertial_cylinder>
     </link>
-    <gazebo reference="back_right_wheel">
+    <gazebo reference="rear_right_wheel">
         <material>Gazebo/Yellow</material>
     </gazebo>
